File: Panelized/carkit PANEL.kicad_pcb (KiCad board)
At the start: 2 copper layers, 100 x 92 mm, 110 parts, among them J1 Barrel_Jack, J10 Conn_02x03_Odd_Even, J11 Conn_01x02_Pin, J12 Conn_01x02_Pin, J2 Conn_01x02_Pin, J3 Conn_02x03_Odd_Even, J4 Conn_02x03_Odd_Even, J5 Conn_01x02_Pin, J6 Conn_01x02_Pin, J7 Barrel_Jack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

Commit message: Panelization Complete
Parts:
- removed H7, H8: MountingHole, MountingHole:MountingHole_3.2mm_M3_Pad_Via
- added G***: LOGO, LOGO, F.Cu at (117.9, 106.2)
- added G***: LOGO, LOGO, B.Cu at (96.0, 122.6)
- added G***: LOGO, LOGO, B.Cu at (129.3, 94.3)
- added G***: LOGO, LOGO, B.Cu at (102.9, 90.8)
- added G***: LOGO, LOGO, B.Cu at (89.3, 99.5)
- added G***: LOGO, LOGO, B.Cu at (119.6, 114.5)
- added G***: LOGO, LOGO, B.Cu at (115.3, 91.4)
- added G***: LOGO, LOGO, B.Cu at (78.9, 118.2)
- added G***1: LOGO, LOGO, B.Cu at (96.0, 70.6)
- added G***2: LOGO, LOGO, B.Cu at (78.9, 66.2)
- added G***3: LOGO, LOGO, B.Cu at (119.6, 62.5)
- added G***4: LOGO, LOGO, F.Cu at (117.9, 54.2)
- added G***5: LOGO, LOGO, B.Cu at (89.3, 47.5)
- added G***6: LOGO, LOGO, B.Cu at (129.3, 42.3)
- added G***7: LOGO, LOGO, B.Cu at (115.3, 39.4)
- added G***8: LOGO, LOGO, B.Cu at (102.9, 38.8)
- moved H4 128.9 mm to (68.9, 75.4)
- moved SW3 72.4 mm to (69.0, 69.2), turned to 180 degrees
- moved SW1 71.6 mm to (69.0, 121.2), turned to 180 degrees
- moved H3 68.5 mm to (127.5, 128.2)
- moved SW4 67.8 mm to (79.5, 76.1), turned to 90 degrees
- moved SW2 67.4 mm to (79.5, 128.1), turned to 90 degrees
- moved C25 67.3 mm to (73.0, 72.5), turned to 180 degrees
- moved C6 66.9 mm to (73.0, 124.5), turned to 180 degrees
- moved R5 66.5 mm to (73.7, 128.8), turned to 90 degrees
- moved R15 66.2 mm to (73.7, 76.8), turned to 90 degrees
- moved C26 64.7 mm to (82.3, 76.1), turned to 90 degrees
- moved C7 64.6 mm to (82.3, 128.1), turned to 90 degrees
- moved R6 61.4 mm to (85.7, 128.1), turned to -90 degrees
- moved R16 61.2 mm to (85.7, 76.1), turned to -90 degrees
- moved D12 58.3 mm to (97.9, 76.4)
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Routing:
- net CHIP_PU: track 82.0 -> 258.3 mm
- net GPIO 9: track 106.3 -> 161.6 mm
- net LED_DATA: track 11.0 -> 62.2 mm
- net GND: track 324.6 -> 284.9 mm, vias 12 -> 18
- net VCC_5V: track 307.2 -> 267.7 mm
- net M2+: track 120.0 -> 85.6 mm, vias 2 -> 6
- net BUZZER_DATA: track 25.9 -> 58.9 mm
- net M2-: track 113.9 -> 87.2 mm, vias 2 -> 6
- net GPIO 8: track 7.21 -> 33.8 mm
- net GPIO 20: track 17.2 -> 34.3 mm
- net GPIO 21: track 22.7 -> 39.6 mm
- net SERVO_PWM: track 67.9 -> 83.4 mm
- net GPIO 10: track 29.3 -> 14.4 mm, vias 4 -> 0
- net D-: track 154.6 -> 142.2 mm
- net D+: track 154.6 -> 142.2 mm
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Other:
- board size 100 x 92 mm -> 75 x 102 mm
- board text added: "10"
- board text added: "20/RX"
- board text added: "21/TX"
- board text added: "Conn."
- board text added: "Drive"
- board text added: "User"
- board text removed: "Connect"
- board text removed: "Drive Motor"
- board text removed: "GPIO10"
- board text removed: "GPIO20 / RX"
- board text removed: "GPIO21 / TX"

Commit message: Quick fix
Parts:
- added SW5: SW_Push, imported_components:SW-SMD_L3.9-W3.0-P4.45, F.Cu at (95.0, 80.4)
- added SW6: SW_SPDT, imported_components:SW-SMD_MST-12D18G4-SPDT-SLIDE-SWITCH, F.Cu at (112.0, 39.2)
- J2, J8: value Conn_01x02_Pin -> Conn_01x02
- SW3: value SW_Push -> SW_SPDT; footprint imported_components:SW-SMD_L3.9-W3.0-P4.45 -> imported_components:SW-SMD_MST-12D18G4-SPDT-SLIDE-SWITCH
- moved SW3 48.4 mm to (112.0, 91.2)
- moved C10 16.0 mm to (137.8, 95.2)
- moved C11 16.0 mm to (118.3, 98.2)
- moved C13 16.0 mm to (114.4, 101.4)
- moved C14 16.0 mm to (111.2, 101.4)
- moved C15 16.0 mm to (125.5, 98.2)
- moved C23 16.0 mm to (112.4, 64.4)
- moved C4 16.0 mm to (112.4, 116.4)
- moved C8 16.0 mm to (137.8, 88.9)
- moved D6 16.0 mm to (113.4, 132.6)
- moved G*** 16.0 mm to (133.4, 110.4)
- moved G*** 16.0 mm to (144.8, 98.5)
- moved G*** 16.0 mm to (135.1, 118.7)
- moved G*** 16.0 mm to (94.4, 122.4)
- moved G***2 16.0 mm to (94.4, 70.4)
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Connections:
- C1 pad 1: +BATT -> REG_BATT+
- C12 pad 1: +BATT -> REG_BATT+
- C13 pad 2: +BATT -> REG_BATT+
- C14 pad 2: +BATT -> REG_BATT+
- C16 pad 1: +BATT -> REG_BATT+
- C17 pad 2: +BATT -> REG_BATT+
- C18 pad 2: +BATT -> REG_BATT+
- C2 pad 2: Net-(U2-VIN) -> REG_BATT+
- C20 pad 1: +BATT -> REG_BATT+
- C21 pad 2: Net-(U2-VIN) -> REG_BATT+
- C31 pad 1: +BATT -> REG_BATT+
- C32 pad 2: +BATT -> REG_BATT+
- C33 pad 2: +BATT -> REG_BATT+
- C35 pad 1: +BATT -> REG_BATT+
- C36 pad 2: +BATT -> REG_BATT+
- C37 pad 2: +BATT -> REG_BATT+
- SW3 pad 1: GPIO 9 -> unconnected-(SW3-A-Pad1)
- SW3 pad 2: GND -> REG_BATT+
- SW4 pad 1: CHIP_PU -> GPIO 9
- U10 pad 11: +BATT -> REG_BATT+
- U2 pad 1: Net-(U2-VIN) -> REG_BATT+
- U4 pad 11: +BATT -> REG_BATT+
- U5 pad 11: +BATT -> REG_BATT+
- U7 pad 1: Net-(U2-VIN) -> REG_BATT+
- U9 pad 11: +BATT -> REG_BATT+
Routing:
- net REG_BATT+: track 0.00 -> 181.7 mm, vias 0 -> 4
- net +BATT: track 182.0 -> 75.7 mm, vias 4 -> 0
- net GND: track 284.9 -> 261.5 mm
- net Net-(U2-VIN): track 8.86 -> 0.00 mm
- net M1-: track 48.5 -> 55.4 mm
- net M1+: track 56.4 -> 62.4 mm
- net CHIP_PU: track 258.3 -> 262.4 mm
- net M2+: track 85.6 -> 82.3 mm
- net LED_DATA: track 62.2 -> 60.9 mm
Other:
- board text added: "OFF"
- board text added: "ON"
