File: PCB/carkit.kicad_sch (KiCad schematic)
At the start: 55 parts, among them J1 Barrel_Jack, J2 Conn_01x02, J3 Conn_02x03_Odd_Even, J4 Conn_02x03_Odd_Even, J5 Conn_01x02_Pin, J6 Conn_01x02_Pin, P1 USB_C_Plug, SW1 SW_Push, SW2 SW_Push, SW3 SW_SPDT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

Commit message: Add CarKit firmware
Added initial CarKit ESP32-C3-MINI firmware which has support for BLE gamepads
Other:
- note added: "Drive Motor"
- note added: "Steering Motor"
Changed lines of the file:
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@@
+		)
+	)
+	(text "Drive Motor"
+		(exclude_from_sim no)
+		(at 233.68 63.246 0)
+		(effects
+			(font
+				(size 1.27 1.27)
+			)
 		)
 	)
@@
 			)
 		)
+	)
+	(text "Steering Motor"
+		(exclude_from_sim no)
+		(at 143.51 62.992 0)
+		(effects
+			(font
+				(size 1.27 1.27)
+			)
+		)
